File: pcb/caninterfaceboard/atmel328pBoard.kicad_sch (KiCad schematic)
At the start: 74 parts, among them J1 UART, J10 NTC2, J12 Flywheel, J13 1Wire, J2 NMEA2000, J3 AVR ISP, J4 NTC3, J5 NTC4, J6 FuelLevel, J7 Engine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

Commit message: Added oil pressure and status, modified pcb
Parts:
- removed C15: 1uF, Capacitor_SMD:C_0805_2012Metric_Pad1.18x1.45mm_HandSolder, symbol Device:C
- removed J2: NMEA2000, Connector_Wire:SolderWire-1.5sqmm_1x04_P6mm_D1.7mm_OD3mm, symbol Connector_Generic:Conn_01x04
- removed J7: Engine, Connector_JST:JST_EH_B4B-EH-A_1x04_P2.50mm_Vertical, symbol Connector_Generic:Conn_01x04
- removed R20: 4.7K, Resistor_SMD:R_0805_2012Metric_Pad1.20x1.40mm_HandSolder, symbol Device:R
- removed R21: 100K, Resistor_SMD:R_0805_2012Metric_Pad1.20x1.40mm_HandSolder, symbol Device:R
- removed SW1: Reset, Button_Switch_SMD:SW_Tactile_SPST_NO_Straight_CK_PTS636Sx25SMTRLFS, symbol Switch:SW_SPST
- added D8: S1J, Diode_SMD:D_0805_2012Metric_Pad1.15x1.40mm_HandSolder, symbol Device:D
- added J2: CAN, TerminalBlock_Phoenix:TerminalBlock_Phoenix_MKDS-1,5-2-5.08_1x02_P5.08mm_Horizontal, symbol Connector_Generic:Conn_01x02
- added J7: Engine, TerminalBlock_Phoenix:TerminalBlock_Phoenix_MKDS-1,5-2-5.08_1x02_P5.08mm_Horizontal, symbol Connector_Generic:Conn_01x02
- added J9: Oil Pressure, TerminalBlock_Phoenix:TerminalBlock_Phoenix_MKDS-1,5-3-5.08_1x03_P5.08mm_Horizontal, symbol Connector_Generic:Conn_01x03
- J1: footprint Connector_PinSocket_2.54mm:PinSocket_1x06_P2.54mm_Horizontal -> Connector_PinSocket_2.54mm:PinSocket_1x06_P2.54mm_Vertical
- J10, J12, J4, J6, J8: footprint Connector_JST:JST_EH_B2B-EH-A_1x02_P2.50mm_Vertical -> TerminalBlock_Phoenix:TerminalBlock_Phoenix_MKDS-1,5-2-5.08_1x02_P5.08mm_Horizontal
- J13: footprint Connector_JST:JST_EH_B3B-EH-A_1x03_P2.50mm_Vertical -> TerminalBlock_Phoenix:TerminalBlock_Phoenix_MKDS-1,5-3-5.08_1x03_P5.08mm_Horizontal
- J5: value NTC4 -> 12V In; footprint Connector_JST:JST_EH_B2B-EH-A_1x02_P2.50mm_Vertical -> TerminalBlock_Phoenix:TerminalBlock_Phoenix_MKDS-1,5-2-5.08_1x02_P5.08mm_Horizontal
Connections:
- net 12V: now also J5.1 (Pin_1)
- net 5V: now also D8.1 (K), J9.1 (Pin_1)
- net A5: now also C19.2, D8.2 (A), J9.2 (Pin_2)
- net Alternator B+: now also J7.1 (Pin_1)
- net CANH: now also J2.2 (Pin_2)
- net CANHL: now also J2.1 (Pin_1)
- net Coolant: now also J7.2 (Pin_2)
- net Engine Batt+: now also C6.1, D7.1 (K), F1.2, U6.3 (VI)
- net GND: now also J9.3 (Pin_3)
Other:
- note added: "Engine Battery"
- note added: "NTC3"
- note added: "Reset pull to gnd. Removed as not used."
- note removed: "12vFused"
- note removed: "Service Battery"
- moved on the sheet: C19
