File: pcb/caninterfaceboard/atmel328pBoard.kicad_sch (KiCad schematic)
At the start: 78 parts, among them J1 AVR UART, J10 NTC2, J11 Attiny UDPI, J12 Flywheel, J13 1Wire, J2 CAN, J3 AVR ISP, J4 NTC3, J5 12V In, J6 FuelLevel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

Commit message: Finally mare the RPM to pulse amp stable
Parts:
- added R13: 1K, Resistor_SMD:R_0805_2012Metric_Pad1.20x1.40mm_HandSolder, symbol Device:R
Connections:
- net 5V: now also R13.2
- net D2: now also R13.1
Other:
- note added: "Internal pullup alone does not provide sufficient current for the open collector in the chip."
- note removed: "Pin configured with pullup"
Changed lines of the file:
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@@
   (junction (at 127.635 52.07) (diameter 0) (color 0 0 0 0)
   )
+  (junction (at 198.755 142.875) (diameter 0) (color 0 0 0 0)
+  )
   (junction (at 46.99 161.925) (diameter 0) (color 0 0 0 0)
   )
@@
   (no_connect (at 59.69 95.885))
   (no_connect (at 59.69 149.225))
+  (wire (pts (xy 198.755 140.97) (xy 198.755 142.875))
+    (stroke (width 0) (type default))
+  )
   (wire (pts (xy 33.655 208.915) (xy 69.85 208.915))
     (stroke (width 0) (type default))
   )
+  (wire (pts (xy 198.755 142.875) (xy 200.66 142.875))
+    (stroke (width 0) (type default))
+  )
   (wire (pts (xy 39.37 180.34) (xy 39.37 175.895))
     (stroke (width 0) (type default))
@@
     (stroke (width 0) (type default))
   )
-  (wire (pts (xy 196.85 142.875) (xy 200.66 142.875))
+  (wire (pts (xy 196.85 142.875) (xy 198.755 142.875))
     (stroke (width 0) (type default))
   )
@@
     (effects (font (size 1.27 1.27)) (justify left bottom))
   )
+  (text "Internal pullup alone does not \nprovide sufficient current for the \nopen collector in the chip."
+    (at 186.69 128.27 0)
+    (effects (font (size 1.27 1.27)) (justify left bottom))
+  )
   (text "CS" (at -72.39 140.335 0)
     (effects (font (size 1.27 1.27)) (justify left bottom))
@@
     (effects (font (size 1.27 1.27)) (justify left bottom))
   )
-  (text "Pin configured with pullup" (at 191.77 131.445 0)
-    (effects (font (size 1.27 1.27)) (justify left bottom))
-  )
   (text "Fuel level" (at 65.405 120.015 0)
     (effects (font (size 1.27 1.27)) (justify left bottom))
@@
     )
   )
+  (global_label "5V" (shape input) (at 198.755 133.35 0) (fields_autoplaced)
+    (effects (font (size 1.27 1.27)) (justify left))
+    (property "Intersheetrefs" "${INTERSHEET_REFS}" (at 204.0383 133.35 0)
+      (effects (font (size 1.27 1.27)) (justify left) hide)
+    )
+  )
   (global_label "5V" (shape input) (at -53.34 158.75 0) (fields_autoplaced)
     (effects (font (size 1.27 1.27)) (justify left))
@@
         )
       )
+    )
+  )
+  (symbol (lib_id "Device:R") (at 198.755 137.16 0) (mirror x) (unit 1)
+    (in_bom yes) (on_board yes) (dnp no) (fields_autoplaced)
+    (property "Reference" "R13" (at 196.85 135.89 0)
+      (effects (font (size 1.27 1.27)) (justify right))
+    )
+    (property "Value" "1K" (at 196.85 138.43 0)
+      (effects (font (size 1.27 1.27)) (justify right))
+    )
+    (property "Footprint" "Resistor_SMD:R_0805_2012Metric_Pad1.20x1.40mm_HandSolder" (at 196.977 137.16 90)
+      (effects (font (size 1.27 1.27)) hide)
+    )
+    (property "Datasheet" "~" (at 198.755 137.16 0)
+      (effects (font (size 1.27 1.27)) hide)
+    )
+    (property "stock" "Y" (at 198.755 137.16 0)
+      (effects (font (size 1.27 1.27)) hide)
+    )
+    (pin "1")
+    (pin "2")
+    (instances
+      (project "atmel328pBoard"
+        (path "/498aeeac-0101-43ba-845f-386b9cebf75b"
+          (reference "R13") (unit 1)
+        )
+      )
